Commit message: CMake corrections

File: urdf/BIM_model.urdf (robot description, URDF)
Before this commit: robot BIM_model, 1 links, 0 joints
Links:
- link bim: geometry collision mesh filename=package://arm_control/urdf/example_building.stl; visual mesh filename=package://arm_control/urdf/example_building.stl

File: urdf/ur.urdf.xacro (robot description, xacro)
@@ -46,5 +46,5 @@
    <xacro:arg name="simulation_controllers" default="" />
    <!-- initial position for simulations (Fake Hardware, Gazebo, Ignition) -->
-   <xacro:arg name="initial_positions_file" default="$(find ur_arm_control)/config/initial_positions.yaml"/>
+   <xacro:arg name="initial_positions_file" default="$(find arm_control)/config/initial_positions.yaml"/>
    <!-- convert to property to use substitution in function -->
    <xacro:property name="initial_positions_file" default="$(arg initial_positions_file)"/>
