Commit message: Refactor UR controller configuration and UI enhancements
- Updated `ur_controllers_namespace.yaml` to replace tf_prefix with "arm_" and adjusted joint names accordingly.
- Enhanced `UI.py` to integrate QTermWidget for terminal functionality alongside status displays in Arm, Base, and Joint Control tabs.
- Modified `position_sender_node.py` to include expected joint names and improved joint state handling.
- Introduced `qtermwidget_wrapper.py` to encapsulate QTermWidget functionality.
- Created `ur_sim_control.launch.py` for improved simulation control and updated `general.launch.py` to reference the new launch file.
- Added wall marker visualization in `planner_node.py` and adjusted cylinder parameters.
- Updated URDF file to remove unnecessary box geometry and added namespace for robot description in Gazebo plugin.

File: urdf/ur.urdf.xacro (robot description, xacro)
@@ -58,14 +58,14 @@
          <origin rpy="0 0 0" xyz="0 0 0"/>
          <geometry>
-           <box size="5 5 0"/>
+           <box size="0 0 0"/>
          </geometry>
-         <material name="ground_white">
+         <!-- <material name="ground_white">
            <color rgba="1 1 1 0.5"/>
-         </material>
+         </material> -->
        </visual>
        <collision>
          <origin rpy="0 0 0" xyz="0 0 0"/>
          <geometry>
-           <box size="5 5 0"/>
+           <box size="0 0 0"/>
          </geometry>
        </collision>
@@ -124,4 +124,8 @@
       <plugin filename="libgazebo_ros2_control.so" name="gazebo_ros2_control">
         <parameters>$(arg simulation_controllers)</parameters>
+        <ros>
+          <namespace>/arm</namespace>
+          <remapping>/robot_description:=/arm/robot_description</remapping>
+        </ros>
       </plugin>
     </gazebo>

Commit message: Reducing arm mass to enable realistic rotation

File: urdf/ur.urdf.xacro (robot description, xacro)
@@ -4,5 +4,5 @@
    <xacro:arg name="name" default="ur"/>
    <!-- import main macro -->
-   <xacro:include filename="$(find ur_description)/urdf/ur_macro.xacro"/>
+   <xacro:include filename="$(find arm_control)/urdf/ur_macro.xacro"/>
    <!-- possible 'ur_type' values: ur3, ur3e, ur5, ur5e, ur10, ur10e, ur16e, ur20, ur30 -->
    <!-- the default value should raise an error in case this was called without defining the type -->
@@ -45,4 +45,5 @@
    <xacro:arg name="sim_ignition" default="false" />
    <xacro:arg name="simulation_controllers" default="" />
+   <xacro:arg name="arm_dyn_scale" default="0.003"/>
    <!-- initial position for simulations (Fake Hardware, Gazebo, Ignition) -->
    <xacro:arg name="initial_positions_file" default="$(find arm_control)/config/initial_positions.yaml"/>
@@ -114,4 +115,5 @@
      script_sender_port="$(arg script_sender_port)"
      trajectory_port="$(arg trajectory_port)"
+     arm_dyn_scale="$(arg arm_dyn_scale)"
      >
      <origin xyz="0 0 0" rpy="0 0 0" />          <!-- position robot in the world -->

File: urdf/ur_macro.xacro (robot description, xacro)
@@ -42,5 +42,6 @@
     trajectory_port:=50003
     non_blocking_read:=true
-    keep_alive_count:=2"
+    keep_alive_count:=2
+    arm_dyn_scale:=0.003"
     >
     <!-- Load configuration data from the provided .yaml files -->
@@ -105,5 +106,5 @@
         </geometry>
       </collision>
-      <xacro:cylinder_inertial radius="${base_inertia_radius}" length="${base_inertia_length}" mass="${base_mass}">
+      <xacro:cylinder_inertial radius="${base_inertia_radius}" length="${base_inertia_length}" mass="${base_mass * arm_dyn_scale}">
         <origin xyz="0 0 0" rpy="0 0 0" />
       </xacro:cylinder_inertial>
@@ -123,13 +124,13 @@
       </collision>
       <inertial>
-        <mass value="${shoulder_mass}"/>
+        <mass value="${shoulder_mass * arm_dyn_scale}"/>
         <origin rpy="${shoulder_inertia_rotation}" xyz="${shoulder_cog}"/>
         <inertia
-            ixx="${shoulder_inertia_ixx}"
-            ixy="${shoulder_inertia_ixy}"
-            ixz="${shoulder_inertia_ixz}"
-            iyy="${shoulder_inertia_iyy}"
-            iyz="${shoulder_inertia_iyz}"
-            izz="${shoulder_inertia_izz}"
+            ixx="${shoulder_inertia_ixx * arm_dyn_scale}"
+            ixy="${shoulder_inertia_ixy * arm_dyn_scale}"
+            ixz="${shoulder_inertia_ixz * arm_dyn_scale}"
+            iyy="${shoulder_inertia_iyy * arm_dyn_scale}"
+            iyz="${shoulder_inertia_iyz * arm_dyn_scale}"
+            izz="${shoulder_inertia_izz * arm_dyn_scale}"
         />
       </inertial>    </link>
@@ -148,13 +149,13 @@
       </collision>
       <inertial>
-        <mass value="${upper_arm_mass}"/>
+        <mass value="${upper_arm_mass * arm_dyn_scale}"/>
         <origin rpy="${upper_arm_inertia_rotation}" xyz="${upper_arm_cog}"/>
         <inertia
-            ixx="${upper_arm_inertia_ixx}"
-            ixy="${upper_arm_inertia_ixy}"
-            ixz="${upper_arm_inertia_ixz}"
-            iyy="${upper_arm_inertia_iyy}"
-            iyz="${upper_arm_inertia_iyz}"
-            izz="${upper_arm_inertia_izz}"
+            ixx="${upper_arm_inertia_ixx * arm_dyn_scale}"
+            ixy="${upper_arm_inertia_ixy * arm_dyn_scale}"
+            ixz="${upper_arm_inertia_ixz * arm_dyn_scale}"
+            iyy="${upper_arm_inertia_iyy * arm_dyn_scale}"
+            iyz="${upper_arm_inertia_iyz * arm_dyn_scale}"
+            izz="${upper_arm_inertia_izz * arm_dyn_scale}"
         />
       </inertial>
@@ -174,13 +175,13 @@
       </collision>
       <inertial>
-        <mass value="${forearm_mass}"/>
+        <mass value="${forearm_mass * arm_dyn_scale}"/>
         <origin rpy="${forearm_inertia_rotation}" xyz="${forearm_cog}"/>
         <inertia
-            ixx="${forearm_inertia_ixx}"
-            ixy="${forearm_inertia_ixy}"
-            ixz="${forearm_inertia_ixz}"
-            iyy="${forearm_inertia_iyy}"
-            iyz="${forearm_inertia_iyz}"
-            izz="${forearm_inertia_izz}"
+            ixx="${forearm_inertia_ixx * arm_dyn_scale}"
+            ixy="${forearm_inertia_ixy * arm_dyn_scale}"
+            ixz="${forearm_inertia_ixz * arm_dyn_scale}"
+            iyy="${forearm_inertia_iyy * arm_dyn_scale}"
+            iyz="${forearm_inertia_iyz * arm_dyn_scale}"
+            izz="${forearm_inertia_izz * arm_dyn_scale}"
         />
       </inertial>
@@ -201,13 +202,13 @@
       </collision>
       <inertial>
-        <mass value="${wrist_1_mass}"/>
+        <mass value="${wrist_1_mass * arm_dyn_scale}"/>
         <origin rpy="${wrist_1_inertia_rotation}" xyz="${wrist_1_cog}"/>
         <inertia
-            ixx="${wrist_1_inertia_ixx}"
-            ixy="${wrist_1_inertia_ixy}"
-            ixz="${wrist_1_inertia_ixz}"
-            iyy="${wrist_1_inertia_iyy}"
-            iyz="${wrist_1_inertia_iyz}"
-            izz="${wrist_1_inertia_izz}"
+            ixx="${wrist_1_inertia_ixx * arm_dyn_scale}"
+            ixy="${wrist_1_inertia_ixy * arm_dyn_scale}"
+            ixz="${wrist_1_inertia_ixz * arm_dyn_scale}"
+            iyy="${wrist_1_inertia_iyy * arm_dyn_scale}"
+            iyz="${wrist_1_inertia_iyz * arm_dyn_scale}"
+            izz="${wrist_1_inertia_izz * arm_dyn_scale}"
         />
       </inertial>
@@ -228,13 +229,13 @@
       </collision>
       <inertial>
-        <mass value="${wrist_2_mass}"/>
+        <mass value="${wrist_2_mass * arm_dyn_scale}"/>
         <origin rpy="${wrist_2_inertia_rotation}" xyz="${wrist_2_cog}"/>
         <inertia
-            ixx="${wrist_2_inertia_ixx}"
-            ixy="${wrist_2_inertia_ixy}"
-            ixz="${wrist_2_inertia_ixz}"
-            iyy="${wrist_2_inertia_iyy}"
-            iyz="${wrist_2_inertia_iyz}"
-            izz="${wrist_2_inertia_izz}"
+            ixx="${wrist_2_inertia_ixx * arm_dyn_scale}"
+            ixy="${wrist_2_inertia_ixy * arm_dyn_scale}"
+            ixz="${wrist_2_inertia_ixz * arm_dyn_scale}"
+            iyy="${wrist_2_inertia_iyy * arm_dyn_scale}"
+            iyz="${wrist_2_inertia_iyz * arm_dyn_scale}"
+            izz="${wrist_2_inertia_izz * arm_dyn_scale}"
         />
       </inertial>
@@ -261,13 +262,13 @@
       </collision>
       <inertial>
-        <mass value="${wrist_3_mass}"/>
+        <mass value="${wrist_3_mass * arm_dyn_scale}"/>
         <origin rpy="${wrist_3_inertia_rotation}" xyz="${wrist_3_cog}"/>
         <inertia
-            ixx="${wrist_3_inertia_ixx}"
-            ixy="${wrist_3_inertia_ixy}"
-            ixz="${wrist_3_inertia_ixz}"
-            iyy="${wrist_3_inertia_iyy}"
-            iyz="${wrist_3_inertia_iyz}"
-            izz="${wrist_3_inertia_izz}"
+            ixx="${wrist_3_inertia_ixx * arm_dyn_scale}"
+            ixy="${wrist_3_inertia_ixy * arm_dyn_scale}"
+            ixz="${wrist_3_inertia_ixz * arm_dyn_scale}"
+            iyy="${wrist_3_inertia_iyy * arm_dyn_scale}"
+            iyz="${wrist_3_inertia_iyz * arm_dyn_scale}"
+            izz="${wrist_3_inertia_izz * arm_dyn_scale}"
         />
       </inertial>

Commit message: Add cylinder adapter between wrist3 and tool0 in URDF. Refactor planner_node and position_sender to take the cylinder into account.

File: urdf/ur.urdf.xacro (robot description, xacro)
@@ -46,4 +46,7 @@
    <xacro:arg name="simulation_controllers" default="" />
    <xacro:arg name="arm_dyn_scale" default="0.003"/>
+   <!-- End-effector cylinder parameters -->
+   <xacro:arg name="ee_cylinder_length" default="0.15"/>
+   <xacro:arg name="ee_cylinder_radius" default="0.035"/>
    <!-- initial position for simulations (Fake Hardware, Gazebo, Ignition) -->
    <xacro:arg name="initial_positions_file" default="$(find arm_control)/config/initial_positions.yaml"/>
@@ -116,4 +119,6 @@
      trajectory_port="$(arg trajectory_port)"
      arm_dyn_scale="$(arg arm_dyn_scale)"
+     ee_cylinder_length="$(arg ee_cylinder_length)"
+     ee_cylinder_radius="$(arg ee_cylinder_radius)"
      >
      <origin xyz="0 0 0" rpy="0 0 0" />          <!-- position robot in the world -->

File: urdf/ur_macro.xacro (robot description, xacro)
@@ -43,5 +43,7 @@
     non_blocking_read:=true
     keep_alive_count:=2
-    arm_dyn_scale:=0.003"
+    arm_dyn_scale:=0.003
+    ee_cylinder_length:=0.15
+    ee_cylinder_radius:=0.035"
     >
     <!-- Load configuration data from the provided .yaml files -->
@@ -396,9 +398,37 @@
       <origin xyz="0 0 0" rpy="0 ${-pi/2.0} ${-pi/2.0}" />
     </joint>
+    <!-- Cylinder adapter between flange and tool0 (parameterized) -->
+    <link name="${tf_prefix}ee_cylinder_link">
+      <visual>
+        <!-- cylinder is centered at this link's origin; URDF cylinders are along local Z,
+             so the joint below rotates 90° around Y to align Z with the flange X-axis -->
+        <origin xyz="0 0 0" rpy="0 0 0"/>
+        <geometry>
+          <cylinder radius="${ee_cylinder_radius}" length="${ee_cylinder_length}"/>
+        </geometry>
+        <material name="ee_cylinder_grey">
+          <color rgba="0.6 0.6 0.6 1.0"/>
+        </material>
+      </visual>
+      <collision>
+        <origin xyz="0 0 0" rpy="0 0 0"/>
+        <geometry>
+          <cylinder radius="${ee_cylinder_radius}" length="${ee_cylinder_length}"/>
+        </geometry>
+      </collision>
+    </link>
+    <!-- Joint: flange -> ee_cylinder_link (centred at half-length along flange X = tool0 Z) -->
+    <joint name="${tf_prefix}flange-ee_cylinder" type="fixed">
+      <parent link="${tf_prefix}flange"/>
+      <child  link="${tf_prefix}ee_cylinder_link"/>
+      <!-- translate half cylinder length along flange X, then rotate 90° around Y so cylinder Z aligns with flange X -->
+      <origin xyz="${ee_cylinder_length / 2.0} 0 0" rpy="0 ${pi/2.0} 0"/>
+    </joint>
     <!-- ROS-Industrial 'tool0' frame - all-zeros tool frame -->
     <link name="${tf_prefix}tool0"/>
     <joint name="${tf_prefix}flange-tool0" type="fixed">
       <!-- default toolframe - X+ left, Y+ up, Z+ front -->
-      <origin xyz="0 0 0" rpy="${pi/2.0} 0 ${pi/2.0}"/>
+      <!-- Full cylinder length offset along flange X (= cylinder length along tool0 Z) -->
+      <origin xyz="${ee_cylinder_length} 0 0" rpy="${pi/2.0} 0 ${pi/2.0}"/>
       <parent link="${tf_prefix}flange"/>
       <child link="${tf_prefix}tool0"/>
