Commit message: Update sensor plate dimensions and adjust end effector cylinder size Adjust collision geometry dimensions for ultrasonic sensor, plate and cylinder

File: urdf/sensor_plate.urdf.xacro (robot description, xacro)
@@ -15,5 +15,5 @@
         <origin xyz="0 0 0" rpy="0 0 0"/>
         <geometry>
-          <box size="0.04 0.04 0.02"/>
+          <box size="0.05 0.05 0.03"/>
         </geometry>
       </collision>
@@ -44,5 +44,5 @@
         <origin xyz="0 0 0" rpy="0 0 0"/>
         <geometry>
-          <box size="0.32 0.32 0.003"/>
+          <box size="0.33 0.33 0.005"/>
         </geometry>
       </collision>

File: urdf/ur_macro.xacro (robot description, xacro)
@@ -414,5 +414,5 @@
         <origin xyz="0 0 0" rpy="0 0 0"/>
         <geometry>
-          <cylinder radius="${ee_cylinder_radius}" length="${ee_cylinder_length}"/>
+          <cylinder radius="${ee_cylinder_radius + 0.01}" length="${ee_cylinder_length}"/>
         </geometry>
       </collision>

Commit message: Add mesh for plate sensor

File: urdf/sensor_plate.urdf.xacro (robot description, xacro)
@@ -66,7 +66,7 @@
     <link name="${tf_prefix}plate_link">
       <visual>
-        <origin xyz="0 0 0" rpy="0 0 0"/>
+        <origin xyz="0 0 0" rpy="-1.57 0 3.14159"/>
         <geometry>
-          <box size="0.32 0.32 0.003"/>
+          <mesh filename="package://navi_wall/navi_wall_description/meshes/sensor_plate.stl" scale="0.001 0.001 0.001"/>
         </geometry>
         <material name="plate_aluminum">
@@ -75,7 +75,7 @@
       </visual>
       <collision>
-        <origin xyz="0 0 0" rpy="0 0 0"/>
+        <origin xyz="0 0 0" rpy="-1.57 0 3.14159"/>
         <geometry>
-          <box size="0.33 0.33 0.005"/>
+          <mesh filename="package://navi_wall/navi_wall_description/meshes/sensor_plate.stl" scale="0.001 0.001 0.001"/>
         </geometry>
       </collision>

Commit message: Fix mesh filename case for sensor plate in URDF

File: urdf/sensor_plate.urdf.xacro (robot description, xacro)
@@ -68,5 +68,5 @@
         <origin xyz="0 0 0" rpy="-1.57 0 3.14159"/>
         <geometry>
-          <mesh filename="package://navi_wall/navi_wall_description/meshes/sensor_plate.stl" scale="0.001 0.001 0.001"/>
+          <mesh filename="package://navi_wall/navi_wall_description/meshes/sensor_plate.STL" scale="0.001 0.001 0.001"/>
         </geometry>
         <material name="plate_aluminum">
@@ -77,5 +77,5 @@
         <origin xyz="0 0 0" rpy="-1.57 0 3.14159"/>
         <geometry>
-          <mesh filename="package://navi_wall/navi_wall_description/meshes/sensor_plate.stl" scale="0.001 0.001 0.001"/>
+          <mesh filename="package://navi_wall/navi_wall_description/meshes/sensor_plate.STL" scale="0.001 0.001 0.001"/>
         </geometry>
       </collision>

Commit message: Update distance sensor configurations: change name for consistency, increase ideal distance and adjust sensor origins

File: urdf/sensor_plate.urdf.xacro (robot description, xacro)
@@ -93,11 +93,11 @@
     <!-- Three ultrasonic sensors -->
     <xacro:ultrasonic_sensor parent_link="${tf_prefix}plate_link" tf_prefix="${tf_prefix}" sensor_name="sensor_A">
-      <origin xyz="-0.15 -0.15 0.005" rpy="0 -1.5708 0"/>
+      <origin xyz="-0.15 -0.15 0.02" rpy="0 -1.5708 0"/>
     </xacro:ultrasonic_sensor>
     <xacro:ultrasonic_sensor parent_link="${tf_prefix}plate_link" tf_prefix="${tf_prefix}" sensor_name="sensor_B">
-      <origin xyz="0.15 -0.15 0.005" rpy="0 -1.5708 0"/>
+      <origin xyz="0.15 -0.15 0.02" rpy="0 -1.5708 0"/>
     </xacro:ultrasonic_sensor>
     <xacro:ultrasonic_sensor parent_link="${tf_prefix}plate_link" tf_prefix="${tf_prefix}" sensor_name="sensor_C">
-      <origin xyz="0 0.15 0.005" rpy="0 -1.5708 0"/>
+      <origin xyz="0 0.15 0.02" rpy="0 -1.5708 0"/>
     </xacro:ultrasonic_sensor>
   </xacro:macro>

Commit message: Add a node to align plate parallel to wall using 6 sensors

File: urdf/sensor_plate.urdf.xacro (robot description, xacro)
@@ -63,4 +63,61 @@
     </gazebo>
   </xacro:macro>
+  <!-- Macro for single ToF sensor (VL6180x). Modeled as a narrow, low-noise,
+       short-range gpu_lidar ray, since Gz Sim has no native ToF type. -->
+  <xacro:macro name="tof_sensor" params="parent_link tf_prefix sensor_name *origin">
+    <link name="${tf_prefix}${sensor_name}_link">
+      <visual>
+        <origin xyz="0 0 0" rpy="-1.57 1.57 0"/>
+        <geometry>
+          <mesh filename="package://navi_wall/navi_wall_description/meshes/ultrasonic.STL" scale="0.0008 0.0008 0.0008"/>
+        </geometry>
+        <material name="tof_red">
+          <color rgba="0.9 0.1 0.1 0.8"/>
+        </material>
+      </visual>
+      <inertial>
+        <mass value="0.003"/>
+        <inertia ixx="1e-6" ixy="0" ixz="0" iyy="1e-6" iyz="0" izz="1e-6"/>
+      </inertial>
+    </link>
+    <joint name="${tf_prefix}${sensor_name}_joint" type="fixed">
+      <parent link="${parent_link}"/>
+      <child link="${tf_prefix}${sensor_name}_link"/>
+      <xacro:insert_block name="origin"/>
+    </joint>
+    <gazebo reference="${tf_prefix}${sensor_name}_link">
+      <sensor name="${sensor_name}_sensor" type="gpu_lidar">
+        <always_on>true</always_on>
+        <update_rate>30</update_rate>
+        <visualize>true</visualize>
+        <topic>/distance_sensors/${sensor_name}</topic>
+        <gz_frame_id>${tf_prefix}${sensor_name}_link</gz_frame_id>
+        <lidar>
+          <scan>
+            <horizontal>
+              <samples>1</samples>
+              <min_angle>-0.0175</min_angle>
+              <max_angle>0.0175</max_angle>
+            </horizontal>
+            <vertical>
+              <samples>1</samples>
+              <min_angle>0</min_angle>
+              <max_angle>0</max_angle>
+            </vertical>
+          </scan>
+          <range>
+            <min>0.01</min>
+            <max>0.18</max>
+            <resolution>0.001</resolution>
+          </range>
+          <noise type="gaussian">
+            <mean>0.0</mean>
+            <stddev>0.002</stddev>
+          </noise>
+        </lidar>
+      </sensor>
+      <self_collide>false</self_collide>
+    </gazebo>
+  </xacro:macro>
   <xacro:macro name="sensor_plate" params="parent_link tf_prefix:='' ee_cylinder_length:=0.15">
     <link name="${tf_prefix}plate_link">
@@ -101,4 +158,14 @@
       <origin xyz="0 0.15 0.02" rpy="0 -1.5708 0"/>
     </xacro:ultrasonic_sensor>
+    <!-- Three ToF sensors (VL6180x): two top corners + one bottom-middle edge -->
+    <xacro:tof_sensor parent_link="${tf_prefix}plate_link" tf_prefix="${tf_prefix}" sensor_name="sensor_D">
+      <origin xyz="0.15 0.15 0.02" rpy="0 -1.5708 0"/>
+    </xacro:tof_sensor>
+    <xacro:tof_sensor parent_link="${tf_prefix}plate_link" tf_prefix="${tf_prefix}" sensor_name="sensor_E">
+      <origin xyz="-0.15 0.15 0.02" rpy="0 -1.5708 0"/>
+    </xacro:tof_sensor>
+    <xacro:tof_sensor parent_link="${tf_prefix}plate_link" tf_prefix="${tf_prefix}" sensor_name="sensor_F">
+      <origin xyz="0 -0.15 0.02" rpy="0 -1.5708 0"/>
+    </xacro:tof_sensor>
   </xacro:macro>
 </robot>

Commit message: Update position of sensors in plate.

File: urdf/sensor_plate.urdf.xacro (robot description, xacro)
@@ -150,21 +150,21 @@
     <!-- Three ultrasonic sensors -->
     <xacro:ultrasonic_sensor parent_link="${tf_prefix}plate_link" tf_prefix="${tf_prefix}" sensor_name="sensor_A">
-      <origin xyz="-0.15 -0.15 0.02" rpy="0 -1.5708 0"/>
+      <origin xyz="-0.155 -0.17 0.02" rpy="0 -1.5708 0"/>
     </xacro:ultrasonic_sensor>
     <xacro:ultrasonic_sensor parent_link="${tf_prefix}plate_link" tf_prefix="${tf_prefix}" sensor_name="sensor_B">
-      <origin xyz="0.15 -0.15 0.02" rpy="0 -1.5708 0"/>
+      <origin xyz="0.155 -0.17 0.02" rpy="0 -1.5708 0"/>
     </xacro:ultrasonic_sensor>
     <xacro:ultrasonic_sensor parent_link="${tf_prefix}plate_link" tf_prefix="${tf_prefix}" sensor_name="sensor_C">
-      <origin xyz="0 0.15 0.02" rpy="0 -1.5708 0"/>
+      <origin xyz="0 0.172 0.02" rpy="0 -1.5708 0"/>
     </xacro:ultrasonic_sensor>
     <!-- Three ToF sensors (VL6180x): two top corners + one bottom-middle edge -->
     <xacro:tof_sensor parent_link="${tf_prefix}plate_link" tf_prefix="${tf_prefix}" sensor_name="sensor_D">
-      <origin xyz="0.15 0.15 0.02" rpy="0 -1.5708 0"/>
+      <origin xyz="0.152 0.17 0.02" rpy="0 -1.5708 0"/>
     </xacro:tof_sensor>
     <xacro:tof_sensor parent_link="${tf_prefix}plate_link" tf_prefix="${tf_prefix}" sensor_name="sensor_E">
-      <origin xyz="-0.15 0.15 0.02" rpy="0 -1.5708 0"/>
+      <origin xyz="-0.152 0.17 0.02" rpy="0 -1.5708 0"/>
     </xacro:tof_sensor>
     <xacro:tof_sensor parent_link="${tf_prefix}plate_link" tf_prefix="${tf_prefix}" sensor_name="sensor_F">
-      <origin xyz="0 -0.15 0.02" rpy="0 -1.5708 0"/>
+      <origin xyz="0 -0.172 0.02" rpy="0 -1.5708 0"/>
     </xacro:tof_sensor>
   </xacro:macro>

Commit message: Fix ToF sensor positions in URDF for consistent layout

File: urdf/sensor_plate.urdf.xacro (robot description, xacro)
@@ -160,8 +160,8 @@
     <!-- Three ToF sensors (VL6180x): two top corners + one bottom-middle edge -->
     <xacro:tof_sensor parent_link="${tf_prefix}plate_link" tf_prefix="${tf_prefix}" sensor_name="sensor_D">
-      <origin xyz="0.152 0.17 0.02" rpy="0 -1.5708 0"/>
+      <origin xyz="-0.152 0.17 0.02" rpy="0 -1.5708 0"/>
     </xacro:tof_sensor>
     <xacro:tof_sensor parent_link="${tf_prefix}plate_link" tf_prefix="${tf_prefix}" sensor_name="sensor_E">
-      <origin xyz="-0.152 0.17 0.02" rpy="0 -1.5708 0"/>
+      <origin xyz="0.152 0.17 0.02" rpy="0 -1.5708 0"/>
     </xacro:tof_sensor>
     <xacro:tof_sensor parent_link="${tf_prefix}plate_link" tf_prefix="${tf_prefix}" sensor_name="sensor_F">

Commit message: Add OAK camera  to sensor plate and update URDF integration

File: urdf/sensor_plate.urdf.xacro (robot description, xacro)
@@ -1,4 +1,5 @@
 <?xml version="1.0"?>
 <robot xmlns:xacro="http://www.ros.org/wiki/xacro">
+  <xacro:include filename="$(find depthai_descriptions_v3)/urdf/include/depthai_macro.urdf.xacro"/>
   <!-- Macro for single ultrasonic sensor -->
   <xacro:macro name="ultrasonic_sensor" params="parent_link tf_prefix sensor_name *origin">
@@ -120,5 +121,16 @@
     </gazebo>
   </xacro:macro>
-  <xacro:macro name="sensor_plate" params="parent_link tf_prefix:='' ee_cylinder_length:=0.15">
+  <xacro:macro name="sensor_plate" params="
+      parent_link
+      tf_prefix:=''
+      ee_cylinder_length:=0.15
+      oak_camera_name:='oak'
+      oak_camera_model:='OAK-D-PRO'
+      oak_cam_pos_x:=0.075
+      oak_cam_pos_y:=0.0
+      oak_cam_pos_z:=0.125
+      oak_cam_roll:=0.0
+      oak_cam_pitch:=-1.5708
+      oak_cam_yaw:=3.14159">
     <link name="${tf_prefix}plate_link">
       <visual>
@@ -168,4 +180,15 @@
       <origin xyz="0 -0.172 0.02" rpy="0 -1.5708 0"/>
     </xacro:tof_sensor>
+    <xacro:depthai_camera
+        camera_name="${oak_camera_name}"
+        camera_model="${oak_camera_model}"
+        parent="${tf_prefix}plate_link"
+        base_frame="${tf_prefix}oak_mount_link"
+        cam_pos_x="${oak_cam_pos_x}"
+        cam_pos_y="${oak_cam_pos_y}"
+        cam_pos_z="${oak_cam_pos_z}"
+        cam_roll="${oak_cam_roll}"
+        cam_pitch="${oak_cam_pitch}"
+        cam_yaw="${oak_cam_yaw}"/>
   </xacro:macro>
 </robot>

File: urdf/ur.urdf.xacro (robot description, xacro)
@@ -51,4 +51,12 @@
    <xacro:arg name="ee_cylinder_radius" default="0.035"/>
    <xacro:arg name="sensors_offset" default="0.15"/>
+   <xacro:arg name="oak_camera_name" default="oak"/>
+   <xacro:arg name="oak_camera_model" default="OAK-D-PRO"/>
+   <xacro:arg name="oak_cam_pos_x" default="0.075"/>
+   <xacro:arg name="oak_cam_pos_y" default="0.0"/>
+   <xacro:arg name="oak_cam_pos_z" default="0.125"/>
+   <xacro:arg name="oak_cam_roll" default="0.0"/>
+   <xacro:arg name="oak_cam_pitch" default="-1.5708"/>
+   <xacro:arg name="oak_cam_yaw" default="3.14159"/>
    <!-- initial position for simulations (Fake Hardware, Gazebo, Ignition) -->
    <xacro:arg name="initial_positions_file" default="$(find arm_control)/config/initial_positions.yaml"/>
@@ -130,5 +138,13 @@
      parent_link="$(arg tf_prefix)ee_cylinder_link"
      tf_prefix="$(arg tf_prefix)"
-     ee_cylinder_length="$(arg ee_cylinder_length)"/>
+     ee_cylinder_length="$(arg ee_cylinder_length)"
+     oak_camera_name="$(arg oak_camera_name)"
+     oak_camera_model="$(arg oak_camera_model)"
+     oak_cam_pos_x="$(arg oak_cam_pos_x)"
+     oak_cam_pos_y="$(arg oak_cam_pos_y)"
+     oak_cam_pos_z="$(arg oak_cam_pos_z)"
+     oak_cam_roll="$(arg oak_cam_roll)"
+     oak_cam_pitch="$(arg oak_cam_pitch)"
+     oak_cam_yaw="$(arg oak_cam_yaw)"/>
    <xacro:if value="$(arg sim_gazebo)">
     <!-- Gazebo Ignition/Gazebo Sim plugins (sim_gazebo now uses Gazebo Ignition, not Classic) -->

Commit message: Update oak camera mount pose to fit REP 103(X-> right, Y-> down, Z->forward)

File: urdf/sensor_plate.urdf.xacro (robot description, xacro)
@@ -132,8 +132,8 @@
       oak_cam_roll:=0.0
       oak_cam_pitch:=-1.5708
-      oak_cam_yaw:=3.14159">
+      oak_cam_yaw:=0">
     <link name="${tf_prefix}plate_link">
       <visual>
-        <origin xyz="0 0 0" rpy="-1.57 0 3.14159"/>
+        <origin xyz="0 0 0" rpy="0 0 0"/>
         <geometry>
           <mesh filename="package://navi_wall/navi_wall_description/meshes/sensor_plate.STL" scale="0.001 0.001 0.001"/>
@@ -144,5 +144,5 @@
       </visual>
       <collision>
-        <origin xyz="0 0 0" rpy="-1.57 0 3.14159"/>
+        <origin xyz="0 0 0" rpy="0 0 0"/>
         <geometry>
           <mesh filename="package://navi_wall/navi_wall_description/meshes/sensor_plate.STL" scale="0.001 0.001 0.001"/>

File: urdf/ur.urdf.xacro (robot description, xacro)
@@ -58,5 +58,5 @@
    <xacro:arg name="oak_cam_roll" default="0.0"/>
    <xacro:arg name="oak_cam_pitch" default="-1.5708"/>
-   <xacro:arg name="oak_cam_yaw" default="3.14159"/>
+   <xacro:arg name="oak_cam_yaw" default="0"/>
    <!-- initial position for simulations (Fake Hardware, Gazebo, Ignition) -->
    <xacro:arg name="initial_positions_file" default="$(find arm_control)/config/initial_positions.yaml"/>
