Commit message: Add tool0 offset from sensors plate

File: srdf/arm_control.srdf.xacro (robot description, xacro)
@@ -43,7 +43,8 @@
   <disable_collisions link1="$(arg tf_prefix)tool0" link2="$(arg tf_prefix)wrist_3_link" reason="Adjacent" />
   <disable_collisions link1="$(arg tf_prefix)ee_cylinder_link" link2="$(arg tf_prefix)wrist_3_link" reason="Never" />
+  <disable_collisions link1="$(arg tf_prefix)tool0" link2="$(arg tf_prefix)plate_link" reason="Adjacent" />
   <disable_collisions link1="$(arg tf_prefix)ee_cylinder_link" link2="$(arg tf_prefix)plate_link" reason="Adjacent" />
-  <disable_collisions link1="$(arg tf_prefix)plate_link" link2="$(arg tf_prefix)sensor_A_sensor_link" reason="Adjacent" />
-  <disable_collisions link1="$(arg tf_prefix)plate_link" link2="$(arg tf_prefix)sensor_B_sensor_link" reason="Adjacent" />
-  <disable_collisions link1="$(arg tf_prefix)plate_link" link2="$(arg tf_prefix)sensor_C_sensor_link" reason="Adjacent" />
+  <disable_collisions link1="$(arg tf_prefix)plate_link" link2="A_link" reason="Adjacent" />
+  <disable_collisions link1="$(arg tf_prefix)plate_link" link2="B_link" reason="Adjacent" />
+  <disable_collisions link1="$(arg tf_prefix)plate_link" link2="C_link" reason="Adjacent" />
 </robot>

File: srdf/mobile_manipulator.srdf.xacro (robot description, xacro)
@@ -51,8 +51,8 @@
   <disable_collisions link1="$(arg tf_prefix)tool0" link2="$(arg tf_prefix)wrist_3_link" reason="Adjacent" />
   <disable_collisions link1="$(arg tf_prefix)ee_cylinder_link" link2="$(arg tf_prefix)wrist_3_link" reason="Never" />
-  <disable_collisions link1="$(arg tf_prefix)tool0" link2="plate_link" reason="Adjacent" />
-  <disable_collisions link1="$(arg tf_prefix)ee_cylinder_link" link2="plate_link" reason="Adjacent" />
-  <disable_collisions link1="plate_link" link2="A_link" reason="Adjacent" />
-  <disable_collisions link1="plate_link" link2="B_link" reason="Adjacent" />
-  <disable_collisions link1="plate_link" link2="C_link" reason="Adjacent" />
+  <disable_collisions link1="$(arg tf_prefix)tool0" link2="$(arg tf_prefix)plate_link" reason="Adjacent" />
+  <disable_collisions link1="$(arg tf_prefix)ee_cylinder_link" link2="$(arg tf_prefix)plate_link" reason="Adjacent" />
+  <disable_collisions link1="$(arg tf_prefix)plate_link" link2="A_link" reason="Adjacent" />
+  <disable_collisions link1="$(arg tf_prefix)plate_link" link2="B_link" reason="Adjacent" />
+  <disable_collisions link1="$(arg tf_prefix)plate_link" link2="C_link" reason="Adjacent" />
 </robot>

File: urdf/sensor_plate.urdf.xacro (robot description, xacro)
@@ -1,34 +1,67 @@
 <?xml version="1.0"?>
 <robot xmlns:xacro="http://www.ros.org/wiki/xacro">
-  <xacro:macro name="sensor_plate_sensor" params="parent_link tf_prefix sensor_name xyz rpy">
-    <link name="${tf_prefix}${sensor_name}_sensor_link">
+  <!-- Macro for single ultrasonic sensor -->
+  <xacro:macro name="ultrasonic_sensor" params="parent_link sensor_name *origin">
+    <link name="${sensor_name}_link">
       <visual>
-        <origin xyz="0 0 0" rpy="0 0 0"/>
+        <origin xyz="0 0 0" rpy="-1.57 1.57 0"/>
         <geometry>
-          <box size="0.04 0.04 0.02"/>
+          <mesh filename="package://navi_wall/navi_wall_description/meshes/ultrasonic.STL" scale="0.001 0.001 0.001"/>
         </geometry>
         <material name="sensor_black">
-          <color rgba="0.05 0.05 0.05 1.0"/>
+          <color rgba="0.0 0.1 0.9 0.8"/>
         </material>
       </visual>
       <collision>
-        <origin xyz="0 0 0" rpy="0 0 0"/>
+        <origin xyz="0 0 0" rpy="-1.57 1.57 0"/>
         <geometry>
-          <box size="0.05 0.05 0.03"/>
+          <mesh filename="package://navi_wall/navi_wall_description/meshes/ultrasonic.STL" scale="0.0015 0.0015 0.0015"/>
         </geometry>
       </collision>
       <inertial>
-        <origin xyz="0 0 0" rpy="0 0 0"/>
         <mass value="0.005"/>
         <inertia ixx="1e-6" ixy="0" ixz="0" iyy="1e-6" iyz="0" izz="1e-6"/>
       </inertial>
     </link>
-    <joint name="${tf_prefix}${sensor_name}_sensor_joint" type="fixed">
+    <joint name="${parent_link}_to_${sensor_name}" type="fixed">
       <parent link="${parent_link}"/>
-      <child link="${tf_prefix}${sensor_name}_sensor_link"/>
-      <origin xyz="${xyz}" rpy="${rpy}"/>
+      <child link="${sensor_name}_link"/>
+      <xacro:insert_block name="origin"/>
     </joint>
+    <gazebo reference="${sensor_name}_link">
+      <sensor name="${sensor_name}_sensor" type="gpu_lidar">
+        <always_on>true</always_on>
+        <update_rate>20</update_rate>
+        <visualize>true</visualize>
+        <topic>/distance_sensors/${sensor_name}</topic>
+        <gz_frame_id>${sensor_name}_link</gz_frame_id>
+        <lidar>
+          <scan>
+            <horizontal>
+              <samples>1</samples>
+              <min_angle>-0.087</min_angle>
+              <max_angle>0.087</max_angle>
+            </horizontal>
+            <vertical>
+              <samples>1</samples>
+              <min_angle>0</min_angle>
+              <max_angle>0</max_angle>
+            </vertical>
+          </scan>
+          <range>
+            <min>0.02</min>
+            <max>4.0</max>
+            <resolution>0.01</resolution>
+          </range>
+          <noise type="gaussian">
+            <mean>0.0</mean>
+            <stddev>0.01</stddev>
+          </noise>
+        </lidar>
+      </sensor>
+      <self_collide>false</self_collide>
+    </gazebo>
   </xacro:macro>
-  <xacro:macro name="sensor_plate" params="parent_link tf_prefix:=''">
+  <xacro:macro name="sensor_plate" params="parent_link tf_prefix:='' ee_cylinder_length:=0.15">
     <link name="${tf_prefix}plate_link">
       <visual>
@@ -56,24 +89,16 @@
       <parent link="${parent_link}"/>
       <child link="${tf_prefix}plate_link"/>
-      <origin xyz="0 0 0" rpy="0 0 0"/>
+      <origin xyz="0 0 ${ee_cylinder_length / 2.0}" rpy="0 0 ${pi/2.0}"/>
     </joint>
-    <xacro:sensor_plate_sensor
-      parent_link="${tf_prefix}plate_link"
-      tf_prefix="${tf_prefix}"
-      sensor_name="sensor_A"
-      xyz="-0.15 -0.15 0.005"
-      rpy="0 -1.5708 0"/>
-    <xacro:sensor_plate_sensor
-      parent_link="${tf_prefix}plate_link"
-      tf_prefix="${tf_prefix}"
-      sensor_name="sensor_B"
-      xyz="0.15 -0.15 0.005"
-      rpy="0 -1.5708 0"/>
-    <xacro:sensor_plate_sensor
-      parent_link="${tf_prefix}plate_link"
-      tf_prefix="${tf_prefix}"
-      sensor_name="sensor_C"
-      xyz="0 0.15 0.005"
-      rpy="0 -1.5708 0"/>
+    <!-- Three ultrasonic sensors -->
+    <xacro:ultrasonic_sensor parent_link="${tf_prefix}plate_link" sensor_name="A">
+      <origin xyz="-0.15 -0.15 0.005" rpy="0 -1.5708 0"/>
+    </xacro:ultrasonic_sensor>
+    <xacro:ultrasonic_sensor parent_link="${tf_prefix}plate_link" sensor_name="B">
+      <origin xyz="0.15 -0.15 0.005" rpy="0 -1.5708 0"/>
+    </xacro:ultrasonic_sensor>
+    <xacro:ultrasonic_sensor parent_link="${tf_prefix}plate_link" sensor_name="C">
+      <origin xyz="0 0.15 0.005" rpy="0 -1.5708 0"/>
+    </xacro:ultrasonic_sensor>
   </xacro:macro>
 </robot>

File: urdf/ur.urdf.xacro (robot description, xacro)
@@ -50,4 +50,5 @@
    <xacro:arg name="ee_cylinder_length" default="0.15"/>
    <xacro:arg name="ee_cylinder_radius" default="0.035"/>
+   <xacro:arg name="sensors_offset" default="0.05"/>
    <!-- initial position for simulations (Fake Hardware, Gazebo, Ignition) -->
    <xacro:arg name="initial_positions_file" default="$(find arm_control)/config/initial_positions.yaml"/>
@@ -122,10 +123,12 @@
      ee_cylinder_length="$(arg ee_cylinder_length)"
      ee_cylinder_radius="$(arg ee_cylinder_radius)"
+     sensors_offset="$(arg sensors_offset)"
      >
      <origin xyz="0 0 0" rpy="0 0 0" />          <!-- position robot in the world -->
    </xacro:ur_robot>
    <xacro:sensor_plate
-     parent_link="$(arg tf_prefix)tool0"
-     tf_prefix="$(arg tf_prefix)"/>
+     parent_link="$(arg tf_prefix)ee_cylinder_link"
+     tf_prefix="$(arg tf_prefix)"
+     ee_cylinder_length="$(arg ee_cylinder_length)"/>
    <xacro:if value="$(arg sim_gazebo)">
     <!-- Gazebo Ignition/Gazebo Sim plugins (sim_gazebo now uses Gazebo Ignition, not Classic) -->

File: urdf/ur_macro.xacro (robot description, xacro)
@@ -45,5 +45,6 @@
     arm_dyn_scale:=0.003
     ee_cylinder_length:=0.15
-    ee_cylinder_radius:=0.035"
+    ee_cylinder_radius:=0.035
+    sensors_offset:=0.05"
     >
     <!-- Load configuration data from the provided .yaml files -->
@@ -427,9 +428,9 @@
     <!-- ROS-Industrial 'tool0' frame - all-zeros tool frame -->
     <link name="${tf_prefix}tool0"/>
-    <joint name="${tf_prefix}flange-tool0" type="fixed">
+    <joint name="${tf_prefix}ee_cylinder-tool0" type="fixed">
       <!-- default toolframe - X+ left, Y+ up, Z+ front -->
       <!-- Full cylinder length offset along flange X (= cylinder length along tool0 Z) -->
-      <origin xyz="${ee_cylinder_length} 0 0" rpy="${pi/2.0} 0 ${pi/2.0}"/>
-      <parent link="${tf_prefix}flange"/>
+      <origin xyz="0 0 ${sensors_offset + ee_cylinder_length / 2.0}" rpy="0 0 ${pi/2.0}"/>
+      <parent link="${tf_prefix}ee_cylinder_link"/>
       <child link="${tf_prefix}tool0"/>
     </joint>

Commit message: Fix bug on legacy mobile-base obstacles disappearing.

File: srdf/arm_control.srdf.xacro (robot description, xacro)
@@ -45,6 +45,6 @@
   <disable_collisions link1="$(arg tf_prefix)tool0" link2="$(arg tf_prefix)plate_link" reason="Adjacent" />
   <disable_collisions link1="$(arg tf_prefix)ee_cylinder_link" link2="$(arg tf_prefix)plate_link" reason="Adjacent" />
-  <disable_collisions link1="$(arg tf_prefix)plate_link" link2="A_link" reason="Adjacent" />
-  <disable_collisions link1="$(arg tf_prefix)plate_link" link2="B_link" reason="Adjacent" />
-  <disable_collisions link1="$(arg tf_prefix)plate_link" link2="C_link" reason="Adjacent" />
+  <disable_collisions link1="$(arg tf_prefix)plate_link" link2="$(arg tf_prefix)sensor_A_link" reason="Adjacent" />
+  <disable_collisions link1="$(arg tf_prefix)plate_link" link2="$(arg tf_prefix)sensor_B_link" reason="Adjacent" />
+  <disable_collisions link1="$(arg tf_prefix)plate_link" link2="$(arg tf_prefix)sensor_C_link" reason="Adjacent" />
 </robot>

File: urdf/sensor_plate.urdf.xacro (robot description, xacro)
@@ -2,6 +2,6 @@
 <robot xmlns:xacro="http://www.ros.org/wiki/xacro">
   <!-- Macro for single ultrasonic sensor -->
-  <xacro:macro name="ultrasonic_sensor" params="parent_link sensor_name *origin">
-    <link name="${sensor_name}_link">
+  <xacro:macro name="ultrasonic_sensor" params="parent_link tf_prefix sensor_name *origin">
+    <link name="${tf_prefix}${sensor_name}_link">
       <visual>
         <origin xyz="0 0 0" rpy="-1.57 1.57 0"/>
@@ -24,10 +24,10 @@
       </inertial>
     </link>
-    <joint name="${parent_link}_to_${sensor_name}" type="fixed">
+    <joint name="${tf_prefix}${sensor_name}_joint" type="fixed">
       <parent link="${parent_link}"/>
-      <child link="${sensor_name}_link"/>
+      <child link="${tf_prefix}${sensor_name}_link"/>
       <xacro:insert_block name="origin"/>
     </joint>
-    <gazebo reference="${sensor_name}_link">
+    <gazebo reference="${tf_prefix}${sensor_name}_link">
       <sensor name="${sensor_name}_sensor" type="gpu_lidar">
         <always_on>true</always_on>
@@ -35,5 +35,5 @@
         <visualize>true</visualize>
         <topic>/distance_sensors/${sensor_name}</topic>
-        <gz_frame_id>${sensor_name}_link</gz_frame_id>
+        <gz_frame_id>${tf_prefix}${sensor_name}_link</gz_frame_id>
         <lidar>
           <scan>
@@ -92,11 +92,11 @@
     </joint>
     <!-- Three ultrasonic sensors -->
-    <xacro:ultrasonic_sensor parent_link="${tf_prefix}plate_link" sensor_name="A">
+    <xacro:ultrasonic_sensor parent_link="${tf_prefix}plate_link" tf_prefix="${tf_prefix}" sensor_name="sensor_A">
       <origin xyz="-0.15 -0.15 0.005" rpy="0 -1.5708 0"/>
     </xacro:ultrasonic_sensor>
-    <xacro:ultrasonic_sensor parent_link="${tf_prefix}plate_link" sensor_name="B">
+    <xacro:ultrasonic_sensor parent_link="${tf_prefix}plate_link" tf_prefix="${tf_prefix}" sensor_name="sensor_B">
       <origin xyz="0.15 -0.15 0.005" rpy="0 -1.5708 0"/>
     </xacro:ultrasonic_sensor>
-    <xacro:ultrasonic_sensor parent_link="${tf_prefix}plate_link" sensor_name="C">
+    <xacro:ultrasonic_sensor parent_link="${tf_prefix}plate_link" tf_prefix="${tf_prefix}" sensor_name="sensor_C">
       <origin xyz="0 0.15 0.005" rpy="0 -1.5708 0"/>
     </xacro:ultrasonic_sensor>
